Commit message: slam_toolbox initial localization completed

File: task4_ws/src/tortoisebot_description/models/tortoisebot_Task4.urdf (robot description, URDF)
Before this commit: robot tortoisebot, 7 links, 6 joints
Joints:
- joint base_joint: origin xyz=0.0 0.0 0.09 rpy=0 0 0 -> xyz=0.0 0.0 0.00 rpy=0 0 0
